File: platypus/hardware/eagle/Old versions/Platypus_v1_0_Proto_v10_0/Platypus.brd (EAGLE design)
At the start: 25.1 x 35.5 mm, 34 parts, among them IC1 MPU-9250, J1 EDISON_CONNECTOR_FULLMOUNTING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, U2 TXS0108E, U3 MAX17043, X1 Power TP, X2 Power TP, X5 Display TP

Commit message: updated platypus hardware folder
Parts:
- removed U$4: TSL25723FNFN-6PIN, TSL25723FN:FN-6PIN
- added U$1: TSL2584TSV6-XFBGA, TSL2584TSV:6-XFBGA
- R3: value 4.7k -> 10k
- moved U$3 3.55 mm to (96.7, 23.4), turned to 270 degrees
Connections:
- net 3.3V: now also U$1.P$1; no longer U$4.P$1
- net ALS_INT: now also U$1.P$5; no longer U$4.P$5
- net GND: now also U$1.P$2, U$1.P$3, U$3.P$5, U$3.P$6; no longer U$3.P$1, U$3.P$2, U$4.P$3
- net GP19_I2C_1_SCL: now also U$1.P$4; no longer U$4.P$2
- net GP20_I2C_1_SDA: now also U$1.P$6; no longer U$4.P$6
- net VSYS: now also U$3.P$1, U$3.P$2; no longer U$3.P$5, U$3.P$6
Routing:
- net GND: track 67.1 -> 73.8 mm
- net ALS_INT: track 9.58 -> 5.95 mm
- net GP20_I2C_1_SDA: track 64.9 -> 62.5 mm
- net 1.8V: track 112.7 -> 114.8 mm
- net 3.3V: track 75.3 -> 76.2 mm
- net GP19_I2C_1_SCL: track 67.3 -> 66.5 mm
Other:
- board text added: "Ambient Light Sensor"
- board text added: "C2 100nF"
- board text added: "C3 100nF"
- board text added: "Prototype v10.0"
- board text added: "R3 10k"
- board text added: "TSL2584TSV"
- board text removed: "Ambient Light Sensor(ALS)"
- board text removed: "C2 0.1µF"
- board text removed: "C3 0.1µF"
- board text removed: "Prototype v11.0"
- board text removed: "R3 4k7"
- board text removed: "TSL25723FN"
