File: platypus/hardware/eagle/Old versions/Platypus_v1_0_Proto_v10_0/Platypus.sch (EAGLE design)
At the start: 34 parts, among them IC1 MPU-9250, J1 EDISON_CONNECTOR_FULLMOUNTING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, U2 TXS0108E, U3 MAX17043, X1 Power TP, X2 Power TP, X5 Display TP

Commit message: updated platypus hardware folder
Parts:
- removed U$4: TSL25723FNFN-6PIN, TSL25723FN:TSL25723FNFN-6PIN
- added U$1: TSL2584TSV6-XFBGA, TSL2584TSV:TSL2584TSV6-XFBGA
- R3: value 4.7k -> 10k
Connections:
- net 3.3V: now also U$1.VDD; no longer U$4.VDD
- net ALS_INT: now also U$1.INT; no longer U$4.INT
- net GND: now also U$1.ADSL, U$1.GND, U$3.P$5, U$3.P$6; no longer U$3.P$1, U$3.P$2, U$4.GND
- net GP19_I2C_1_SCL: now also U$1.SCL; no longer U$4.SCL
- net GP20_I2C_1_SDA: now also U$1.SDA; no longer U$4.SDA
- net VSYS: now also U$3.P$1, U$3.P$2; no longer U$3.P$5, U$3.P$6
Other:
- moved on the sheet: C7, R12
