File: platypus/hardware/eagle/Old versions/Platypus_v1_0_Proto_v12_0/Platypus.brd (EAGLE design)
At the start: 25.1 x 35.5 mm, 34 parts, among them IC1 MPU-9250, J1 EDISON_CONNECTOR_FULLMOUNTING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, U2 TXS0108E, U3 MAX17043, X1 Power TP, X2 Power TP, X5 Display TP

Commit message: updated platypus hardware folder
Parts:
- removed U$4: TSL25723FNFN-6PIN, TSL25723FN:FN-6PIN
- added C9: 100nF, Discrete:C0603
- added IC2: MCP73831, microchip-update-2:SOT23-5L
- added R13: 1k, Discrete:R0603
- added R14: 10k, Discrete:R0603
- added TP1, TP2: PTR1TP19SQ, testpad:TP19SQ
- added U$1: TSL2584TSV6-XFBGA, TSL2584TSV:6-XFBGA
- R3: value 4.7k -> 10k
- moved U$3 3.55 mm to (96.7, 23.4), turned to 270 degrees
- moved R3 1.31 mm to (94.7, 14.6), turned to 0 degrees
- moved C2 1.15 mm to (94.8, 16.8)
- moved C8 0.63 mm to (89.8, 37.9)
- moved R9 0.50 mm to (90.1, 27.5)
- moved C_VCCB 0.39 mm to (90.1, 34.6), turned to 90 degrees
- moved C_VCCA 0.10 mm to (90.1, 31.6)
Connections:
- removed net GP19_I2C_1_SCL: IC1.23, J1.41, R6.1, U$4.P$2, U3.7, X1.4
- removed net GP20_I2C_1_SDA: IC1.24, J1.43, R5.1, U$4.P$6, U3.8, X1.2
- new net N$10: C9.2, IC2.4, TP2.TP
- new net N$2: IC2.5, R13.2
- net 1.8V: now also R14.2
- net 3.3V: now also U$1.P$1; no longer U$4.P$1
- net ALS_INT: now also U$1.P$5; no longer U$4.P$5
- net GND: now also C9.1, IC2.2, R13.1, TP1.TP, U$1.P$2, U$1.P$3, U$3.P$5, U$3.P$6; no longer U$3.P$1, U$3.P$2, U$4.P$3
- net GP27_I2C_6_SCL: now also IC1.23, R6.1, U$1.P$4, U3.7, X1.4
- net GP28_I2C_6_SDA: now also IC1.24, R5.1, U$1.P$6, U3.8, X1.2
- net GP45: now also IC2.1, R14.1
- net VSYS: now also IC2.3, U$3.P$1, U$3.P$2; no longer U$3.P$5, U$3.P$6
Routing:
- net GP19_I2C_1_SCL: track 67.3 -> 0.00 mm, vias 7 -> 0
- net GP27_I2C_6_SCL: track 0.00 -> 66.6 mm, vias 0 -> 7
- net GP20_I2C_1_SDA: track 64.9 -> 0.00 mm, vias 10 -> 0
- net GP28_I2C_6_SDA: track 0.00 -> 61.4 mm, vias 0 -> 7
- net GP45: track 0.00 -> 23.6 mm, vias 0 -> 2
- net GND: track 67.1 -> 75.7 mm, vias 9 -> 14
- net 1.8V: track 112.7 -> 119.4 mm
- net N$10: track 0.00 -> 4.16 mm
- net VSYS: track 47.1 -> 51.2 mm, vias 5 -> 6
- net ALS_INT: track 9.58 -> 5.95 mm
- net 3.3V: track 75.3 -> 78.5 mm
- net N$2: track 0.00 -> 2.02 mm
- net N$9: track 0.50 -> 2.34 mm
- net IMU_INT: track 24.9 -> 23.2 mm
- net GP44: track 17.7 -> 17.5 mm, vias 4 -> 2
Other:
- board text added: "Ambient Light Sensor"
- board text added: "C2 100nF"
- board text added: "C3 100nF"
- board text added: "Prototype v10.0"
- board text added: "R3 10k"
- board text added: "TSL2584TSV"
- board text removed: "Ambient Light Sensor(ALS)"
- board text removed: "C2 0.1µF"
- board text removed: "C3 0.1µF"
- board text removed: "Prototype v11.0"
- board text removed: "R3 4k7"
- board text removed: "TSL25723FN"
