File: platypus/hardware/eagle/Old versions/Platypus_v1_0_Proto_v12_0/Platypus.sch (EAGLE design)
At the start: 27 parts, among them J1 EDISON_CONNECTOR_FULLMOUNTING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, U1 MPU-9250, U2 TXB0108, U3 MAX17043, X3 Power TP, X4 I2C TP, X5 Display TP

Commit message: updated platypus hardware folder
Parts:
- removed R2, R4: 10k, Discrete:R-0603
- removed U1: MPU-9250, template:MPU-9150
- removed X3: Power TP, con-molex:53047-04
- removed X4: I2C TP, con-molex:53047-06
- added C3, C9: 100nF, Discrete:C-0603
- added C7: 0.1µF, Discrete:C-0603
- added IC1: MPU-9250, invensense:MPU-9250
- added IC2: MCP73831, microchip-update-2:MCP73831
- added INT_J3: (no value), jumper:SJ
- added R10, R11, R12: 4.7k, Discrete:R-0603
- added R13: 1k, Discrete:R-0603
- added R14: 10k, Discrete:R-0603
- added TP1, TP2: PTR1TP19SQ, testpad:PTR1TP19SQ
- added U$1: TSL2584TSV6-XFBGA, TSL2584TSV:TSL2584TSV6-XFBGA
- added U$2: BME280LGA-8, BME280:BME280LGA-8
- added U$3: HIROSE_BAT_CON, Hirose_Bat_Con:HIROSE_BAT_CON
- added X1, X2: Power TP, con-molex:53047-04
- U2: value TXB0108 -> TXS0108E
Connections:
- removed net GP19_I2C_1_SCL: J1.GP19_I2C_1_SCL, R6.1, U3.SCL, X4-5.S
- removed net GP20_I2C_1_SDA: J1.GP20_I2C_1_SDA, R5.1, U3.SDA, X4-4.S
- new net ALS_INT: INT_J3.1, R12.1, U$1.INT
- new net AUX_CL: IC1.AUX_CL, R11.1, U$2.SCK
- new net AUX_DA: IC1.AUX_DA, R10.1, U$2.SDI
- new net N$10: C9.2, IC2.VDD, TP2.TP
- new net N$2: IC2.PROG, R13.2
- new net N$8: U2.B4, X-4.1
- new net N$9: U$3.P$3, U$3.P$4
- net 1.8V: now also C3.2, IC1.!CS, IC1.VCC@1, IC1.VCCIO, R10.2, R11.2, R12.2, R14.2, U$2.CSB, U$2.SDO, U$2.VDD, U$2.VDDL, X2-3.S; no longer R2.1, R4.2, U1.CLKIN, U1.CLKOUT, U1.VLOGIC, X3-3.S
- net 3.3V: now also C7.2, IC1.VCC@2, U$1.VDD, X2-2.S; no longer U1.VDD@1, X-4.1, X3-2.S
- net BAT_ALERT: now also X1-3.S; no longer X4-6.S
- net GND: now also C3.1, C7.1, C9.1, IC1.AD0/SDO, IC1.FSYNC, IC1.GND@1, IC1.GND@2, IC2.VSS, R13.1, TP1.TP, U$1.ADSL, U$1.GND, U$2.GND1, U$2.GND2, U$3.P$5, U$3.P$6, X2-4.S; no longer U1.AD0, U1.CPOUT, U1.FSYNC, U1.GND@2, X3-4.S
- net GP27_I2C_6_SCL: now also IC1.SCL/SCLK, R6.1, U$1.SCL, U3.SCL, X1-4.S; no longer R2.2, U1.SCL\, X4-2.S
- net GP28_I2C_6_SDA: now also IC1.SDA/SDI, R5.1, U$1.SDA, U3.SDA, X1-2.S; no longer R4.1, U1.SDA, X4-1.S
- net GP44: now also U2.A4
- net GP45: now also IC2.STAT, R14.1
- net GP80_SD_0_DAT0: now also INT_J3.2
- net IMU_INT: now also IC1.INT, X1-1.S; no longer U1.INT, X4-3.S
- net N$5: now also IC1.REGOUT; no longer U1.REGOUT
- net VSYS: now also IC2.VBAT, U$3.P$1, U$3.P$2, X2-1.S; no longer X3-1.S
Other:
- note added: "Battery Connector"
- moved on the sheet: C1, C2, C4, C5, C6, C8, C_VCCA, C_VCCB, INT_J1, INT_J2, R3, R5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
