File: platypus/hardware/eagle/Old versions/Platypus_v1_0_Proto_v5_0/Platypus_v1_0_Proto_v5_0.brd (EAGLE design)
At the start: 25.1 x 35.5 mm, 27 parts, among them IC1 MPU-9250, J1 EDISON_CONNECTOR_FULLMOUNTING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, U2 TXB0108, U3 MAX17043, X3 Power TP, X4 I2C TP, X5 Display TP

Commit message: updated platypus hardware folder
Parts:
- added INT_J3: (no value), jumper:SJ
- added U$1: TSL2584TSV6-XFBGA, TSL2584TSV:6-XFBGA
- U2: value TXB0108 -> TXS0108E
Connections:
- new net ALS_INT: INT_J3.1, U$1.P$5
- net 3.3V: now also U$1.P$1
- net GND: now also U$1.P$2, U$1.P$3
- net GP19_I2C_1_SCL: now also U$1.P$4
- net GP20_I2C_1_SDA: now also U$1.P$6
- net GP80_SD_0_DAT0: now also INT_J3.2
Routing:
- net GP80_SD_0_DAT0: track 0.00 -> 32.5 mm, vias 0 -> 4
- net GP20_I2C_1_SDA: track 23.7 -> 55.6 mm, vias 4 -> 8
- net GP19_I2C_1_SCL: track 29.3 -> 56.0 mm, vias 3 -> 5
- net 3.3V: track 58.4 -> 69.9 mm
- net GND: track 77.9 -> 86.9 mm, vias 2 -> 3
- net ALS_INT: track 0.00 -> 7.63 mm
- net VSYS: track 36.9 -> 37.9 mm
Other:
- board text added: "Ambient Light Sensor"
- board text added: "J_ALS"
- board text added: "Prototype v5.0"
- board text added: "TSL2584TSV"
- board text added: "TXS0108E"
- board text removed: "Prototype v4.0"
- board text removed: "TXB0108"
