File: platypus/hardware/eagle/Old versions/Platypus_v1_0_Proto_v5_0/Platypus_v1_0_Proto_v5_0.sch (EAGLE design)
At the start: 28 parts, among them J1 EDISON_CONNECTOR_FULLMOUNTING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, U1 MPU-9150, U2 TXB0108, U3 MAX17043, X3 Power TP, X4 I2C TP, X5 Display TP

Commit message: updated platypus hardware folder
Parts:
- removed C3: 2.2nF, Discrete:C-0603
- removed U1: MPU-9150, template:MPU-9150
- added IC1: MPU-9250, invensense:MPU-9250
- added INT_J3: (no value), jumper:SJ
- added U$1: TSL2584TSV6-XFBGA, TSL2584TSV:TSL2584TSV6-XFBGA
- U2: value TXB0108 -> TXS0108E
Connections:
- removed net N$2: C3.2, U1.CPOUT
- new net ALS_INT: INT_J3.1, U$1.INT
- net 1.8V: now also IC1.!CS, IC1.VCC@1, IC1.VCCIO; no longer U1.VLOGIC
- net 3.3V: now also IC1.VCC@2, U$1.VDD; no longer U1.VDD, U1.VDD@1
- net GND: now also IC1.AD0/SDO, IC1.FSYNC, IC1.GND@1, IC1.GND@2, U$1.ADSL, U$1.GND; no longer C3.1, U1.AD0, U1.CLKIN, U1.FSYNC, U1.GND, U1.GND@1, U1.GND@2
- net GP19_I2C_1_SCL: now also U$1.SCL
- net GP20_I2C_1_SDA: now also U$1.SDA
- net GP27_I2C_6_SCL: now also IC1.SCL/SCLK; no longer U1.SCL\
- net GP28_I2C_6_SDA: now also IC1.SDA/SDI; no longer U1.SDA
- net GP80_SD_0_DAT0: now also INT_J3.2
- net IMU_INT: now also IC1.INT; no longer U1.INT
- net N$5: now also IC1.REGOUT; no longer U1.REGOUT
Other:
- moved on the sheet: C1, C2, C4, C5, C6, INT_J1, INT_J2, R2, R3, R4, R5, R6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
