File: platypus/hardware/eagle/Old versions/Platypus_v1_0_Proto_v8_0/Platypus_v1_0_Proto_v8_0.brd (EAGLE design)
At the start: 25.1 x 35.5 mm, 34 parts, among them IC1 MPU-9250, J1 EDISON_CONNECTOR_FULLMOUNTING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, U2 TXS0108E, U3 MAX17043, X1 Power TP, X2 Power TP, X5 Display TP

Commit message: updated platypus hardware folder
Parts:
- removed U$3: HIROSE_BAT_CON, Hirose_Bat_Con:0.5MM-PITCH,6-PIN
- removed U$4: TSL25723FNFN-6PIN, TSL25723FN:FN-6PIN
- removed X1, X2: Power TP, con-molex:53047-04
- added R2, R4: 10k, Discrete:R0603
- added U$1: TSL2584TSV6-XFBGA, TSL2584TSV:6-XFBGA
- added X3: Power TP, con-molex:53047-04
- added X4: I2C TP, con-molex:53047-06
- R3: value 4.7k -> 10k
- moved INT_J3 8.61 mm to (92.8, 33.2)
- moved R12 3.50 mm to (92.8, 38.4), turned to 90 degrees
- moved C3 1.68 mm to (85.2, 17.5)
- moved R1 0.48 mm to (85.2, 22.9)
Connections:
- removed net N$8: U2.16, X.4
- removed net N$9: U$3.P$3, U$3.P$4
- net 1.8V: now also R2.1, R4.2, X3.3; no longer X2.3
- net 3.3V: now also U$1.P$1, X3.2; no longer U$4.P$1, X2.2
- net ALS_INT: now also U$1.P$5; no longer U$4.P$5
- net BAT_ALERT: now also X4.6; no longer X1.3
- net GND: now also U$1.P$2, U$1.P$3, X3.4; no longer U$3.P$1, U$3.P$2, U$4.P$3, X2.4
- net GP19_I2C_1_SCL: now also U$1.P$4, X4.5; no longer IC1.23, U$4.P$2, X1.4
- net GP20_I2C_1_SDA: now also U$1.P$6, X4.4; no longer IC1.24, U$4.P$6, X1.2
- net GP27_I2C_6_SCL: now also IC1.23, R2.2, X4.2
- net GP28_I2C_6_SDA: now also IC1.24, R4.1, X4.1
- net GP44: now also X.4; no longer U2.5
- net IMU_INT: now also X4.3; no longer X1.1
- net VSYS: now also X3.1; no longer U$3.P$5, U$3.P$6, X2.1
Routing:
- net GP28_I2C_6_SDA: track 0.00 -> 34.4 mm, vias 0 -> 3
- net GP27_I2C_6_SCL: track 0.00 -> 28.9 mm, vias 0 -> 4
- net GP80_SD_0_DAT0: track 39.8 -> 27.6 mm
- net GP19_I2C_1_SCL: track 67.3 -> 55.9 mm, vias 7 -> 5
- net GP20_I2C_1_SDA: track 64.9 -> 55.6 mm, vias 10 -> 8
- net VSYS: track 47.1 -> 38.6 mm, vias 5 -> 3
- net N$8: track 7.89 -> 0.00 mm
- net 3.3V: track 75.3 -> 70.0 mm
- net GP44: track 17.7 -> 22.4 mm, vias 4 -> 2
- net GND: track 67.1 -> 71.7 mm, vias 9 -> 7
- net ALS_INT: track 9.58 -> 13.0 mm
- net 1.8V: track 112.7 -> 109.8 mm, vias 7 -> 6
- net BAT_ALERT: track 24.4 -> 22.1 mm
- net N$9: track 0.50 -> 0.00 mm
Other:
- board text added: "Ambient Light Sensor"
- board text added: "BAT_SCL"
- board text added: "BAT_SDA"
- board text added: "C2 100nF"
- board text added: "C3 100nF"
- board text added: "IMU_SCL"
- board text added: "IMU_SDA"
- board text added: "Power Test Point"
- board text added: "Prototype v8.0"
- board text added: "R2 10k"
- board text added: "R3 10k"
- board text added: "R4 10k"
- board text added: "TSL2584TSV"
- board text removed: "Ambient Light Sensor(ALS)"
- board text removed: "C2 0.1µF"
- board text removed: "C3 0.1µF"
- board text removed: "I2C_1_SCL"
- board text removed: "I2C_1_SDA"
- board text removed: "Power Connector"
- board text removed: "Power TP"
- board text removed: "Prototype v11.0"
- board text removed: "R3 4k7"
- board text removed: "TEMP"
- board text removed: "TSL25723FN"
